File: HL_TX-RX_Filter.sch (KiCad schematic (older format))
At the start: 199 parts, among them J1 CNR1, J10 To Rx in, J11 CONN_01X03, J2 CNR3, J3 Antenna, J4 CNR2, J5 CNR4, J6 From Tx, J7 ICSP, J8 CONN_01X05, J9 SCL SDA, Q1 2N7002, Q2 2N7002, Q3 2N7002, Q4 2N7002, Q5 2N7002, Q6 2N7002, Q7 2N7002, Q8 2N7002, U1 ATMEGA328-AU, U10 PE4259, U11 PE4259, U12 PE4259, U2 PE4259, U3 PE4259, U4 PE4259, U5 PE4259, U6 PE4259, U7 PE4259, U8 PE4259, U9 PE4259

Commit message: Changed to Bourns chokes and progressed layout
Parts:
- added C44: 0.1u, Capacitors_SMD:C_1206_HandSoldering, symbol C
- L10, L22, L23, L24: value Choke -> L; footprint Inductors_G:BalunCoreChoke -> Inductors_G:L_1812_HandSoldering
- L11, L12, L13, L14, L20, L3, L9: footprint Inductors_G:BalunCoreChoke -> Inductors_G:L_1812_HandSoldering
Connections:
- wire segments 369 -> 370
Changed lines of the file:
@@
 F 0 "L14" V 3250 6775 50  0000 C CNN
 F 1 "L" V 3375 6775 50  0000 C CNN
-F 2 "Inductors_G:BalunCoreChoke" H 3300 6775 50  0001 C CNN
+F 2 "Inductors_G:L_1812_HandSoldering" H 3300 6775 50  0001 C CNN
 F 3 "" H 3300 6775 50  0001 C CNN
 	1    3300 6775
@@
 F 0 "L3" V 1900 6850 50  0000 C CNN
 F 1 "L" V 2025 6850 50  0000 C CNN
-F 2 "Inductors_G:BalunCoreChoke" H 1950 6850 50  0001 C CNN
+F 2 "Inductors_G:L_1812_HandSoldering" H 1950 6850 50  0001 C CNN
 F 3 "" H 1950 6850 50  0001 C CNN
 	1    1950 6850
@@
 F 0 "L20" V 4500 6775 50  0000 C CNN
 F 1 "L" V 4625 6775 50  0000 C CNN
-F 2 "Inductors_G:BalunCoreChoke" H 4550 6775 50  0001 C CNN
+F 2 "Inductors_G:L_1812_HandSoldering" H 4550 6775 50  0001 C CNN
 F 3 "" H 4550 6775 50  0001 C CNN
 	1    4550 6775
@@
 F 0 "L13" V 3250 5675 50  0000 C CNN
 F 1 "L" V 3375 5675 50  0000 C CNN
-F 2 "Inductors_G:BalunCoreChoke" H 3300 5675 50  0001 C CNN
+F 2 "Inductors_G:L_1812_HandSoldering" H 3300 5675 50  0001 C CNN
 F 3 "" H 3300 5675 50  0001 C CNN
 	1    3300 5675
@@
 F 0 "L12" V 3250 4575 50  0000 C CNN
 F 1 "L" V 3375 4575 50  0000 C CNN
-F 2 "Inductors_G:BalunCoreChoke" H 3300 4575 50  0001 C CNN
+F 2 "Inductors_G:L_1812_HandSoldering" H 3300 4575 50  0001 C CNN
 F 3 "" H 3300 4575 50  0001 C CNN
 	1    3300 4575
@@
 F 0 "L11" V 3250 3475 50  0000 C CNN
 F 1 "L" V 3375 3475 50  0000 C CNN
-F 2 "Inductors_G:BalunCoreChoke" H 3300 3475 50  0001 C CNN
+F 2 "Inductors_G:L_1812_HandSoldering" H 3300 3475 50  0001 C CNN
 F 3 "" H 3300 3475 50  0001 C CNN
 	1    3300 3475
@@
 P 3300 2375
 F 0 "L10" V 3250 2375 50  0000 C CNN
-F 1 "Choke" V 3375 2375 50  0000 C CNN
-F 2 "Inductors_G:BalunCoreChoke" H 3300 2375 50  0001 C CNN
+F 1 "L" V 3375 2375 50  0000 C CNN
+F 2 "Inductors_G:L_1812_HandSoldering" H 3300 2375 50  0001 C CNN
 F 3 "" H 3300 2375 50  0001 C CNN
 	1    3300 2375
@@
 F 0 "L9" V 3250 1275 50  0000 C CNN
 F 1 "L" V 3375 1275 50  0000 C CNN
-F 2 "Inductors_G:BalunCoreChoke" H 3300 1275 50  0001 C CNN
+F 2 "Inductors_G:L_1812_HandSoldering" H 3300 1275 50  0001 C CNN
 F 3 "" H 3300 1275 50  0001 C CNN
 	1    3300 1275
@@
 P 7000 1575
 F 0 "L24" V 7075 1675 50  0000 C CNN
-F 1 "Choke" V 6925 1600 50  0000 C CNN
-F 2 "Inductors_G:BalunCoreChoke" H 7000 1575 50  0001 C CNN
+F 1 "L" V 6925 1600 50  0000 C CNN
+F 2 "Inductors_G:L_1812_HandSoldering" H 7000 1575 50  0001 C CNN
 F 3 "" H 7000 1575 50  0001 C CNN
 	1    7000 1575
@@
 P 5675 1575
 F 0 "L22" V 5750 1650 50  0000 C CNN
-F 1 "Choke" V 5600 1600 50  0000 C CNN
-F 2 "Inductors_G:BalunCoreChoke" H 5675 1575 50  0001 C CNN
+F 1 "L" V 5600 1600 50  0000 C CNN
+F 2 "Inductors_G:L_1812_HandSoldering" H 5675 1575 50  0001 C CNN
 F 3 "" H 5675 1575 50  0001 C CNN
 	1    5675 1575
@@
 P 6450 2075
 F 0 "L23" V 6400 2075 50  0000 C CNN
-F 1 "Choke" V 6525 2075 50  0000 C CNN
-F 2 "Inductors_G:BalunCoreChoke" H 6450 2075 50  0001 C CNN
+F 1 "L" V 6525 2075 50  0000 C CNN
+F 2 "Inductors_G:L_1812_HandSoldering" H 6450 2075 50  0001 C CNN
 F 3 "" H 6450 2075 50  0001 C CNN
 	1    6450 2075
@@
 Connection ~ 3300 1125
 Wire Wire Line
-	1025 4950 1950 4950
+	1025 4950 1300 4950
+Wire Wire Line
+	1600 4950 1950 4950
 Connection ~ 1950 4950
 Wire Wire Line
@@
 	6800 7650 6800 6350
 Wire Bus Line
-	7600 6350 6800 6350
+	6800 6350 7600 6350
 Wire Bus Line
-	7600 5450 7600 6350
+	7600 6350 7600 5450
 Wire Wire Line
 	4575 900  3725 900
@@
 Wire Wire Line
 	6600 2075 6675 2075
+$Comp
+L C C44
+U 1 1 597F3EBC
+P 1450 4950
+F 0 "C44" V 1525 5050 50  0000 L CNN
+F 1 "0.1u" V 1525 4725 50  0000 L CNN
+F 2 "Capacitors_SMD:C_1206_HandSoldering" H 1488 4800 50  0001 C CNN
+F 3 "" H 1450 4950 50  0001 C CNN
+	1    1450 4950
+	0    -1   -1   0
+$EndComp
 $EndSCHEMATC

Commit message: Add Tx/Rx changeover components
Parts:
- added R22, R34, R35: 680, Resistors_SMD:R_1206_HandSoldering, symbol R
- R1, R18, R19, R2, R20, R21, R25, R3, R4: value R -> 680
Connections:
- net labels added: BiasV
- wire segments 370 -> 374
Other:
- moved on the sheet: C46, L23, R25, R26
Changed lines of the file:
@@
 P 1950 7175
 F 0 "R4" V 2030 7175 50  0000 C CNN
-F 1 "R" V 1950 7175 50  0000 C CNN
+F 1 "680" V 1950 7175 50  0000 C CNN
 F 2 "Resistors_SMD:R_1206_HandSoldering" V 1880 7175 50  0001 C CNN
 F 3 "" H 1950 7175 50  0001 C CNN
@@
 P 4475 7075
 F 0 "R19" V 4555 7075 50  0000 C CNN
-F 1 "R" V 4475 7075 50  0000 C CNN
+F 1 "680" V 4475 7075 50  0000 C CNN
 F 2 "Resistors_SMD:R_1206_HandSoldering" V 4405 7075 50  0001 C CNN
 F 3 "" H 4475 7075 50  0001 C CNN
@@
 L C C46
 U 1 1 58F5DE13
-P 6800 750
-F 0 "C46" H 6825 850 50  0000 L CNN
-F 1 "0.1u" H 6825 650 50  0000 L CNN
-F 2 "Capacitors_SMD:C_1206_HandSoldering" H 6838 600 50  0001 C CNN
-F 3 "" H 6800 750 50  0001 C CNN
-	1    6800 750
+P 6675 750
+F 0 "C46" H 6700 850 50  0000 L CNN
+F 1 "0.1u" H 6700 650 50  0000 L CNN
+F 2 "Capacitors_SMD:C_1206_HandSoldering" H 6713 600 50  0001 C CNN
+F 3 "" H 6675 750 50  0001 C CNN
+	1    6675 750
 	1    0    0    -1
 $EndComp
@@
 L GND #PWR034
 U 1 1 58F5DE19
-P 6800 900
-F 0 "#PWR034" H 6800 650 50  0001 C CNN
-F 1 "GND" H 6800 750 50  0001 C CNN
-F 2 "" H 6800 900 50  0001 C CNN
-F 3 "" H 6800 900 50  0001 C CNN
-	1    6800 900
+P 6675 900
+F 0 "#PWR034" H 6675 650 50  0001 C CNN
+F 1 "GND" H 6675 750 50  0001 C CNN
+F 2 "" H 6675 900 50  0001 C CNN
+F 3 "" H 6675 900 50  0001 C CNN
+	1    6675 900
 	1    0    0    -1
 $EndComp
@@
 P 6575 1575
 F 0 "D23" H 6575 1675 50  0000 C CNN
-F 1 "M7" H 6575 1475 50  0000 C CNN
+F 1 "M7" H 6500 1475 50  0000 C CNN
 F 2 "Diodes_SMD:D_SMA_Handsoldering" H 6575 1575 50  0001 C CNN
 F 3 "" H 6575 1575 50  0001 C CNN
@@
 L R R26
 U 1 1 591588BA
-P 7325 1300
-F 0 "R26" V 7405 1300 50  0000 C CNN
-F 1 "R" V 7325 1300 50  0000 C CNN
-F 2 "Resistors_SMD:R_1206_HandSoldering" V 7255 1300 50  0001 C CNN
-F 3 "" H 7325 1300 50  0001 C CNN
-	1    7325 1300
+P 7325 850
+F 0 "R26" V 7405 850 50  0000 C CNN
+F 1 "R" V 7325 850 50  0000 C CNN
+F 2 "Resistors_SMD:R_1206_HandSoldering" V 7255 850 50  0001 C CNN
+F 3 "" H 7325 850 50  0001 C CNN
+	1    7325 850
 	-1   0    0    1
 $EndComp
@@
 L R R25
 U 1 1 591A7757
-P 6225 1800
-F 0 "R25" V 6305 1800 50  0000 C CNN
-F 1 "R" V 6225 1800 50  0000 C CNN
-F 2 "Resistors_SMD:R_1206_HandSoldering" V 6155 1800 50  0001 C CNN
-F 3 "" H 6225 1800 50  0001 C CNN
-	1    6225 1800
-	-1   0    0    1
+P 6450 2125
+F 0 "R25" V 6530 2125 50  0000 C CNN
+F 1 "680" V 6450 2125 50  0000 C CNN
+F 2 "Resistors_SMD:R_1206_HandSoldering" V 6380 2125 50  0001 C CNN
+F 3 "" H 6450 2125 50  0001 C CNN
+	1    6450 2125
+	0    -1   -1   0
 $EndComp
 $Comp
 L L L23
 U 1 1 591A80A2
-P 6450 2075
-F 0 "L23" V 6400 2075 50  0000 C CNN
-F 1 "L" V 6525 2075 50  0000 C CNN
-F 2 "Inductors_G:L_1812_HandSoldering" H 6450 2075 50  0001 C CNN
-F 3 "" H 6450 2075 50  0001 C CNN
-	1    6450 2075
-	0    1    1    0
+P 6225 1800
+F 0 "L23" V 6300 1800 50  0000 C CNN
+F 1 "L" V 6175 1725 50  0000 C CNN
+F 2 "Inductors_G:L_1812_HandSoldering" H 6225 1800 50  0001 C CNN
+F 3 "" H 6225 1800 50  0001 C CNN
+	1    6225 1800
+	-1   0    0    1
 $EndComp
 $Comp
@@
 	1    0    0    -1
 $EndComp
-Text GLabel 6675 2075 2    60   Input ~ 0
-3V3
+Text GLabel 6675 2050 2    60   Input ~ 0
+BiasV
 Text GLabel 7900 2675 0    60   Input ~ 0
 3V3
@@
 P 1775 7175
 F 0 "R3" V 1855 7175 50  0000 C CNN
-F 1 "R" V 1775 7175 50  0000 C CNN
+F 1 "680" V 1775 7175 50  0000 C CNN
 F 2 "Resistors_SMD:R_1206_HandSoldering" V 1705 7175 50  0001 C CNN
 F 3 "" H 1775 7175 50  0001 C CNN
@@
 P 1600 7175
 F 0 "R2" V 1680 7175 50  0000 C CNN
-F 1 "R" V 1600 7175 50  0000 C CNN
+F 1 "680" V 1600 7175 50  0000 C CNN
 F 2 "Resistors_SMD:R_1206_HandSoldering" V 1530 7175 50  0001 C CNN
 F 3 "" H 1600 7175 50  0001 C CNN
@@
 P 1425 7175
 F 0 "R1" V 1505 7175 50  0000 C CNN
-F 1 "R" V 1425 7175 50  0000 C CNN
+F 1 "680" V 1425 7175 50  0000 C CNN
 F 2 "Resistors_SMD:R_1206_HandSoldering" V 1355 7175 50  0001 C CNN
 F 3 "" H 1425 7175 50  0001 C CNN
@@
 P 4650 7075
 F 0 "R20" V 4730 7075 50  0000 C CNN
-F 1 "R" V 4650 7075 50  0000 C CNN
+F 1 "680" V 4650 7075 50  0000 C CNN
 F 2 "Resistors_SMD:R_1206_HandSoldering" V 4580 7075 50  0001 C CNN
 F 3 "" H 4650 7075 50  0001 C CNN
@@
 P 4300 7075
 F 0 "R18" V 4380 7075 50  0000 C CNN
-F 1 "R" V 4300 7075 50  0000 C CNN
+F 1 "680" V 4300 7075 50  0000 C CNN
 F 2 "Resistors_SMD:R_1206_HandSoldering" V 4230 7075 50  0001 C CNN
 F 3 "" H 4300 7075 50  0001 C CNN
@@
 P 4825 7075
 F 0 "R21" V 4905 7075 50  0000 C CNN
-F 1 "R" V 4825 7075 50  0000 C CNN
+F 1 "680" V 4825 7075 50  0000 C CNN
 F 2 "Resistors_SMD:R_1206_HandSoldering" V 4755 7075 50  0001 C CNN
 F 3 "" H 4825 7075 50  0001 C CNN
@@
 Connection ~ 5950 1575
 Wire Wire Line
-	7325 1450 7325 2025
+	7325 1000 7325 2025
 Wire Wire Line
 	6725 1575 6850 1575
@@
 Wire Wire Line
 	3725 900  3725 600
-Connection ~ 6800 600
+Connection ~ 6675 600
 Connection ~ 3725 900
 Wire Wire Line
@@
 Connection ~ 6225 1575
 Wire Wire Line
-	7325 600  7325 1150
+	7325 600  7325 700
 Wire Wire Line
 	4575 1575 4550 1575
@@
 	7700 4600 7900 4600
 Wire Wire Line
-	6225 1950 6225 2075
-Wire Wire Line
-	6225 2075 6300 2075
+	6225 1950 6225 2050
 Wire Wire Line
-	6600 2075 6675 2075
+	6225 2050 6300 2050
 $Comp
 L C C44
@@
 	0    -1   -1   0
 $EndComp
+$Comp
+L R R35
+U 1 1 59800CA0
+P 6450 2300
+F 0 "R35" V 6530 2300 50  0000 C CNN
+F 1 "680" V 6450 2300 50  0000 C CNN
+F 2 "Resistors_SMD:R_1206_HandSoldering" V 6380 2300 50  0001 C CNN
+F 3 "" H 6450 2300 50  0001 C CNN
+	1    6450 2300
+	0    -1   -1   0
+$EndComp
+$Comp
+L R R34
+U 1 1 59801186
+P 6450 1950
+F 0 "R34" V 6530 1950 50  0000 C CNN
+F 1 "680" V 6450 1950 50  0000 C CNN
+F 2 "Resistors_SMD:R_1206_HandSoldering" V 6380 1950 50  0001 C CNN
+F 3 "" H 6450 1950 50  0001 C CNN
+	1    6450 1950
+	0    -1   -1   0
+$EndComp
+$Comp
+L R R22
+U 1 1 598013FE
+P 6450 1775
+F 0 "R22" V 6530 1775 50  0000 C CNN
+F 1 "680" V 6450 1775 50  0000 C CNN
+F 2 "Resistors_SMD:R_1206_HandSoldering" V 6380 1775 50  0001 C CNN
+F 3 "" H 6450 1775 50  0001 C CNN
+	1    6450 1775
+	0    -1   -1   0
+$EndComp
+Wire Wire Line
+	6300 1775 6300 2300
+Connection ~ 6300 1950
+Connection ~ 6300 2050
+Connection ~ 6300 2125
+Wire Wire Line
+	6600 1775 6600 2300
+Connection ~ 6600 1950
+Connection ~ 6600 2125
+Wire Wire Line
+	6675 2050 6600 2050
+Connection ~ 6600 2050
+Text GLabel 4225 7400 0    60   Input ~ 0
+BiasV
+Wire Wire Line
+	4225 7400 4300 7400
+Wire Wire Line
+	4300 7400 4300 7500
+Connection ~ 4300 7500
 $EndSCHEMATC

Commit message: More layout around bias voltage area
Parts:
- added C75: .1u, Capacitors_SMD:C_1206_HandSoldering, symbol C
- added D30, D31, D32, D33: M7, Diodes_SMD:D_SMA, symbol D
- added J12: + - 12v, Pin_Headers:Pin_Header_Straight_1x02_Pitch2.54mm, symbol CONN_01X02
Connections:
- net labels added: +12v
- net labels removed: +12V
- wire segments 374 -> 384
